File: KiCad/circuit-schema/circuit-schema.kicad_sch (KiCad schematic)
At the start: 0 parts

Commit message: kicad MCP added and schema building started
Parts:
- added R1: 10k, symbol project-symbols:R
- added RV1: 10k, symbol project-symbols:R_POT
- added U1: NodeMCU_12E, symbol project-symbols:NodeMCU_12E_ESP8266
- added U2: AM2302, symbol project-symbols:AM2302
- added U3: WC1602A, symbol project-symbols:WC1602A
Connections:
- new net +3V3: R1.2, U1.5 (SD2/GPIO9), U2.3 (NC)
- new net +5V: RV1.3, U1.1 (A0)
- new net DHT_DATA: R1.1, U1.12 (EN), U2.2 (SDA)
- new net GND: RV1.1, U1.17 (D1/GPIO5), U1.2 (RSV), U1.24 (D6/GPIO12), U1.6 (SD1/MOSI), U3.16 (LED-)
- new net LCD_DB4: U1.27 (RX/GPIO3)
- new net LCD_DB5: U1.26 (D8/GPIO15)
- new net LCD_DB6: U1.23 (D5/GPIO14)
- new net LCD_DB7: U1.22 (GND)
- new net LCD_E: U1.28 (TX/GPIO1)
- new net LCD_RS: U1.29 (GND)
- new net LCD_V0: RV1.2
Changed lines of the file:
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@@
-(kicad_sch
-	(version 20260306)
-	(generator "eeschema")
-	(generator_version "10.0")
-	(paper "A4")
-	(sheet_instances
-		(path "/"
-			(page "1")
-		)
-	)
-	(embedded_fonts no)
-)
